Commit message: 20260201: complete:xacro

File: src/aicar_simulation/urdf/aicar.urdf.xacro (robot description, xacro)
@@ -66,6 +66,25 @@
                 </geometry>
             </visual>
+            <!-- 添加碰撞属性 -->
+            <collision>
+                <geometry>
+                    <cylinder radius="${wheel_radius}" length="${wheel_width}" />
+                </geometry>
+            </collision>
             <xacro:cylinder_inertia m="2.0" r="${wheel_radius}" h="${wheel_width}" />
         </link>
+        <!-- 添加摩擦系数 -->
+        <gazebo reference="{prefix}_link">
+            <!-- 摩擦系数 -->
+            <mu1 value="1.0" /> <!-- 滚动方向的摩擦力(主方向) -->
+            <mu2 value="1.0" /> <!-- 与滚动方向垂直的摩擦力(侧向) -->
+            <!-- 接触刚度与阻尼 -->
+            <kp value="10000000.0" /> <!-- 接触刚度：决定轮子有多“硬”。值越大，越不容易陷进地里 -->
+            <kd value="1.0" />        <!-- 接触阻尼：决定轮子碰到地时的“弹性”。值太小，车会像蹦床一样乱跳 -->
+            <!-- 摩擦力方向 -->
+            <fdir1 value="1 0 0" /> <!-- 定义摩擦力的主方向。1 0 0 表示沿 X 轴 -->
+            <!-- 颜色 -->
+            <material>Gazebo/Black</material>  <!-- 在 Gazebo 里给轮子涂上黑色 -->
+        </gazebo>
         <joint name="${prefix}_joint" type="continuous">
             <parent link="base_link" />
@@ -89,3 +108,42 @@
     <xacro:wheel prefix="rear_left" x_reflect="-1" y_reflect="1" />
     <xacro:wheel prefix="rear_right" x_reflect="-1" y_reflect="-1" />
+    <!-- 10. Gazebo差速驱动插件 -->
+    <gazebo>
+        <plugin name='diff_drive' filename='libgazebo_ros_diff_drive.so'>
+            <!-- ROS 节点配置：定义话题名称 -->
+            <ros>
+                <!-- 将内部默认话题重映射为标准的 cmd_vel (控制指令) 和 odom (里程计) -->
+                <remapping>cmd_vel:=cmd_vel</remapping>
+                <remapping>odom:=odom</remapping>
+            </ros>
+            <!-- 轮子关节数量 -->
+            <!-- 2 代表有两对轮子（一共4个轮子）。插件会把左侧两个绑在一起，右侧两个绑在一起 -->
+            <num_wheel_pairs>2</num_wheel_pairs>
+            <!-- 驱动关节配置：必须与你上面 wheel 宏生成的 joint 名字完全一致 -->
+            <left_joint>front_left_joint</left_joint>
+            <left_joint>rear_left_joint</left_joint> <!-- 四轮车可以写多对 -->
+            <right_joint>front_right_joint</right_joint>
+            <right_joint>rear_right_joint</right_joint>
+            <!-- 物理尺寸：这直接影响速度计算的准确性 -->
+            <!-- 轮距：左右轮子中心点的距离（计算转向的关键） -->
+            <wheel_separation>${car_width + wheel_width}</wheel_separation>
+            <!-- 轮子直径：计算前进速度的关键 -->
+            <wheel_diameter>${2 * wheel_radius}</wheel_diameter>
+            <!-- 力矩-->
+            <max_wheel_torque>500</max_wheel_torque>
+            <!-- 最大加速度：值越大，起步越快，但太大会导致车头“翘头”或原地打滑 -->
+            <max_wheel_acceleration>1.0</max_wheel_acceleration>
+            <!-- 输出 -->
+            <!-- 是否发布里程计数据 (Odometry) -->
+            <publish_odom>true</publish_odom>
+            <!-- 是否发布从 odom 到 base_footprint 的坐标变换 (TF) -->
+            <publish_odom_tf>true</publish_odom_tf>
+            <!-- 是否发布轮子的坐标变换（这样 Rviz 里能看到轮子在转） -->
+            <publish_wheel_tf>true</publish_wheel_tf>
+            <!-- 里程计坐标系(TF)的名字。它代表机器人运动的“起始点”参考系，通常固定设为 odom -->
+            <odomery_frame>odom</odomery_frame>
+            <!-- 机器人的根坐标系 -->
+            <robot_base_frame>base_footprint</robot_base_frame>
+        </plugin>
+    </gazebo>
 </robot>

Commit message: feat:20260204,ackermann底盘仿真车搭建成功！

File: src/aicar_simulation/urdf/aicar.urdf.xacro (robot description, xacro)
@@ -8,4 +8,8 @@
     <xacro:property name="wheel_width" default="0.1" />
     <xacro:property name="wheel_radius" default="0.18" />
+    <!-- 新增：前后轮轴心到车体中心的距离 -->
+    <xacro:property name="axle_offset" default="0.5" />
+    <!-- 修正轴距公式：前轴到后轴的距离 -->
+    <xacro:property name="wheel_base" default="${2 * axle_offset}" />
     <!-- 3.离地间隙 -->
     <xacro:property name="clearance" default="0.10" />
@@ -16,7 +20,7 @@
             <mass value="${m}" />
             <inertia
-                ixx="${(m/12) * (h*h + d*d)}" ixy="0.0" ixz="0.0"
-                iyy="${(m/12) * (w*w + d*d)}" iyz="0.0"
-                izz="${(m/12) * (w*w + h*h)}" />
+                ixx="${(m/12) * (w*w + h*h)}" ixy="0.0" ixz="0.0"
+                iyy="${(m/12) * (d*d + h*h)}" iyz="0.0"
+                izz="${(m/12) * (w*w + d*d)}" />
         </inertial>
     </xacro:macro>
@@ -49,6 +53,19 @@
             </geometry>
         </collision>
-        <xacro:box_inertia m="200.0" w="${car_width}" h="${car_height}" d="${car_length}" />
+        <xacro:box_inertia m="20.0" w="${car_width}" h="${car_height}" d="${car_length}" />
     </link>
+    <!-- 舵机驱动 link （虚拟的转向杆） -->
+    <link name="steer_link">
+        <inertial>
+            <mass value="1.0" />
+            <inertia ixx="0.01" ixy="0.0" ixz="0.0" iyy="0.01" iyz="0.0" izz="0.01" />
+        </inertial>
+    </link>
+    <joint name="steer_joint" type="fixed">
+        <parent link="base_link" />
+        <child link="steer_link" />
+        <!-- 放在前轴的中心点，用于计算转向几何 -->
+        <origin xyz="0.0 0.0 0.0" rpy="0.0 0.0 0.0" />
+    </joint>
     <!-- 7.关节:把车身驾在 Footprint 上 -->
     <joint name="base_joint" type="fixed">
@@ -58,90 +75,126 @@
         <origin xyz="0.0 0.0 ${car_height/2 + clearance}" rpy="0.0 0.0 0.0" />
     </joint>
-    <!-- 8.轮子宏 -->
-    <xacro:macro name="wheel" params="prefix x_reflect y_reflect">
-        <link name="${prefix}_link">
+    <!-- 后轮宏：只有滚动 -->
+    <xacro:macro name="rear_wheel" params="prefix x_reflect y_reflect">
+        <link name="${prefix}_wheel_link">
             <visual>
+                <origin xyz="0.0 0.0 0.0" rpy="${pi/2} 0.0 0.0" />
                 <geometry>
                     <cylinder radius="${wheel_radius}" length="${wheel_width}" />
                 </geometry>
             </visual>
-            <!-- 添加碰撞属性 -->
             <collision>
+                <origin xyz="0.0 0.0 0.0" rpy="${pi/2} 0.0 0.0" />
                 <geometry>
                     <cylinder radius="${wheel_radius}" length="${wheel_width}" />
                 </geometry>
             </collision>
-            <xacro:cylinder_inertia m="2.0" r="${wheel_radius}" h="${wheel_width}" />
+            <xacro:cylinder_inertia m="3.0" r="${wheel_radius}" h="${wheel_width}" />
         </link>
-        <!-- 添加摩擦系数 -->
-        <gazebo reference="${prefix}_link">
-            <!-- 摩擦系数 -->
-            <mu1 value="1.0" /> <!-- 滚动方向的摩擦力(主方向) -->
-            <mu2 value="0.01" /> <!-- 与滚动方向垂直的摩擦力(侧向) -->
-            <!-- 接触刚度与阻尼 -->
-            <kp value="10000000.0" /> <!-- 接触刚度：决定轮子有多“硬”。值越大，越不容易陷进地里 -->
-            <kd value="1.0" />        <!-- 接触阻尼：决定轮子碰到地时的“弹性”。值太小，车会像蹦床一样乱跳 -->
-            <!-- 摩擦力方向 -->
-            <fdir1 value="1 0 0" /> <!-- 定义摩擦力的主方向。1 0 0 表示沿 X 轴 -->
-            <!-- 颜色 -->
-            <material>Gazebo/Black</material>  <!-- 在 Gazebo 里给轮子涂上黑色 -->
-        </gazebo>
-        <joint name="${prefix}_joint" type="continuous">
+        <joint name="${prefix}_wheel_joint" type="continuous">
             <parent link="base_link" />
-            <child link="${prefix}_link" />
-            <!--
-               通用位置计算公式：
-               X: 车长的一半 * 系数。这里减 0.1 是为了让轮子不装在车头最顶端，稍微往里收一点(轴距)。
-               Y: 车宽的一半 + 轮子宽度的一半 -> 保证轮子紧贴车身侧面，不多不少。
-               Z: 轮子半径 - (离地间隙 + 车高的一半) -> 自动计算轮轴相对于车身中心的垂直偏移。
-            -->
+            <child link="${prefix}_wheel_link" />
             <origin
                 xyz="${x_reflect * (car_length/2 - 0.1)} ${y_reflect * (car_width/2 + wheel_width/2)} ${wheel_radius - (clearance + car_height/2)}"
-                rpy="${-pi/2} 0 0" />
-            <!-- 绕哪个轴转? 因为上面 rpy 已经把 Z 轴转成指向侧面了,所以这里还是绕 Z 转 -->
+                rpy="0 0 0" />
+            <axis xyz="0 1 0" />
+        </joint>
+        <gazebo reference="${prefix}_wheel_link">
+            <mu1>1.0</mu1>
+            <mu2>1.0</mu2>
+            <kp>1000000.0</kp>
+            <kd>1.0</kd>
+        </gazebo>
+    </xacro:macro>
+    <!-- 前轮宏：可以转向和滚动 -->
+    <xacro:macro name="front_wheel" params="prefix x_reflect y_reflect">
+        <!-- 转向节link -->
+        <link name="${prefix}_steering_hinge">
+            <xacro:cylinder_inertia m="0.1" r="0.05" h="0.05" />
+        </link>
+        <!-- 转向关节：绕Z轴旋转 -->
+        <joint name="${prefix}_steering_joint" type="revolute">
+            <parent link="base_link" />
+            <child link="${prefix}_steering_hinge" />
+            <origin
+                xyz="${x_reflect * (car_length/2 - 0.1)} ${y_reflect * (car_width/2 + wheel_width/2)} ${wheel_radius - (clearance + car_height/2)}"
+                rpy="0.0 0.0 0.0" />
             <axis xyz="0 0 1" />
+            <limit lower="-0.5235" upper="0.5235" effort="1000.0" velocity="100.0" />
+            <!-- 增加以下这行：damping 是阻尼，friction 是静态摩擦 -->
+            <dynamics damping="10.0" friction="1.0" />
         </joint>
+        <!-- 轮子link -->
+        <link name="${prefix}_wheel_link">
+            <visual>
+                <origin xyz="0.0 0.0 0.0" rpy="${pi/2} 0.0 0.0" />
+                <geometry>
+                    <cylinder radius="${wheel_radius}" length="${wheel_width}" />
+                </geometry>
+            </visual>
+            <collision>
+                <origin xyz="0.0 0.0 0.0" rpy="${pi/2} 0.0 0.0" />
+                <geometry>
+                    <cylinder radius="${wheel_radius}" length="${wheel_width}" />
+                </geometry>
+            </collision>
+            <xacro:cylinder_inertia m="3.0" r="${wheel_radius}" h="${wheel_width}" />
+        </link>
+        <!-- 轮子滚动关节： 绕y轴旋转 -->
+        <joint name="${prefix}_wheel_joint" type="continuous">
+            <parent link="${prefix}_steering_hinge" />
+            <child link="${prefix}_wheel_link" />
+            <axis xyz="0 1 0" />
+        </joint>
+        <gazebo reference="${prefix}_wheel_link">
+            <mu1>1.0</mu1>
+            <mu2>1.0</mu2>
+            <kp>1000000.0</kp>
+            <kd>10.0</kd>
+        </gazebo>
     </xacro:macro>
     <!-- 9.调用宏生成4个轮子 -->
-    <xacro:wheel prefix="front_left" x_reflect="1" y_reflect="1" />
-    <xacro:wheel prefix="front_right" x_reflect="1" y_reflect="-1" />
-    <xacro:wheel prefix="rear_left" x_reflect="-1" y_reflect="1" />
-    <xacro:wheel prefix="rear_right" x_reflect="-1" y_reflect="-1" />
-    <!-- 10. Gazebo差速驱动插件 -->
+    <xacro:front_wheel prefix="front_left" x_reflect="1" y_reflect="1" />
+    <xacro:front_wheel prefix="front_right" x_reflect="1" y_reflect="-1" />
+    <xacro:rear_wheel prefix="rear_left" x_reflect="-1" y_reflect="1" />
+    <xacro:rear_wheel prefix="rear_right" x_reflect="-1" y_reflect="-1" />
+    <!-- 10. Gazebo阿克曼驱动插件 -->
     <gazebo>
-        <plugin name='diff_drive' filename='libgazebo_ros_diff_drive.so'>
-            <!-- ROS 节点配置：定义话题名称 -->
+        <plugin name="ackermann_drive" filename="libgazebo_ros_ackermann_drive.so">
             <ros>
-                <!-- 将内部默认话题重映射为标准的 cmd_vel (控制指令) 和 odom (里程计) -->
-                <remapping>cmd_vel:=cmd_vel</remapping>
-                <remapping>odom:=odom</remapping>
+                <!-- 推荐在ROS 2 Humble中使用精确的话题重映射 -->
+                <remapping>cmd_vel:=/cmd_vel</remapping>
+                <remapping>odom:=/odom</remapping>
             </ros>
-            <!-- 轮子关节数量 -->
-            <!-- 2 代表有两对轮子（一共4个轮子）。插件会把左侧两个绑在一起，右侧两个绑在一起 -->
-            <num_wheel_pairs>2</num_wheel_pairs>
-            <!-- 驱动关节配置：必须与你上面 wheel 宏生成的 joint 名字完全一致 -->
-            <left_joint>front_left_joint</left_joint>
-            <left_joint>rear_left_joint</left_joint> <!-- 四轮车可以写多对 -->
-            <right_joint>front_right_joint</right_joint>
-            <right_joint>rear_right_joint</right_joint>
-            <!-- 物理尺寸：这直接影响速度计算的准确性 -->
-            <!-- 轮距：左右轮子中心点的距离（计算转向的关键） -->
+            <update_rate>100.0</update_rate>
+            <!-- 关节名称 -->
+            <!-- 转向关节 -->
+            <left_steering_joint>front_left_steering_joint</left_steering_joint>
+            <right_steering_joint>front_right_steering_joint</right_steering_joint>
+            <!-- 驱动关节: 这里我们将驱动也放在前轮上，阿克曼模型通常是前轮转向、后轮驱动或四轮驱动 -->
+            <!-- 如果您希望是后轮驱动，请确保模型物理属性和PID参数适应这种情况 -->
+            <front_left_joint>front_left_wheel_joint</front_left_joint>
+            <front_right_joint>front_right_wheel_joint</front_right_joint>
+            <rear_left_joint>rear_left_wheel_joint</rear_left_joint>
+            <rear_right_joint>rear_right_wheel_joint</rear_right_joint>
+            <!-- 几何参数 -->
             <wheel_separation>${car_width + wheel_width}</wheel_separation>
-            <!-- 轮子直径：计算前进速度的关键 -->
             <wheel_diameter>${2 * wheel_radius}</wheel_diameter>
-            <!-- 力矩-->
-            <max_wheel_torque>500</max_wheel_torque>
-            <!-- 最大加速度：值越大，起步越快，但太大会导致车头“翘头”或原地打滑 -->
-            <max_wheel_acceleration>1.0</max_wheel_acceleration>
+            <!-- 轴距的计算是前后轮转向轴中心的距离，您的计算是正确的 -->
+            <wheel_base>${2 * (car_length/2 - 0.1)}</wheel_base>
+            <!-- 限制参数 -->
+            <max_steer>0.5235</max_steer>
+            <max_speed>20.0</max_speed>
+            <!-- PID增益 -->
+            <left_steering_pid_gain>4000 0.5 50</left_steering_pid_gain>
+            <right_steering_pid_gain>4000 0.5 50</right_steering_pid_gain>
+            <!-- 驱动 PID： 后驱重点给这两个 -->
+            <linear_velocity_pid_gain>50 0 0</linear_velocity_pid_gain>
             <!-- 输出 -->
-            <!-- 是否发布里程计数据 (Odometry) -->
             <publish_odom>true</publish_odom>
-            <!-- 是否发布从 odom 到 base_footprint 的坐标变换 (TF) -->
             <publish_odom_tf>true</publish_odom_tf>
-            <!-- 是否发布轮子的坐标变换（这样 Rviz 里能看到轮子在转） -->
             <publish_wheel_tf>true</publish_wheel_tf>
-            <!-- 里程计坐标系(TF)的名字。它代表机器人运动的“起始点”参考系，通常固定设为 odom -->
-            <odomery_frame>odom</odomery_frame>
-            <!-- 机器人的根坐标系 -->
+            <publish_distance>true</publish_distance>
+            <odometry_frame>odom</odometry_frame>
             <robot_base_frame>base_footprint</robot_base_frame>
         </plugin>

Commit message: feat: 20260206 添加雷达以及imu后

File: src/aicar_simulation/urdf/aicar.urdf.xacro (robot description, xacro)
@@ -200,3 +200,170 @@
         </plugin>
     </gazebo>
+    <!-- 感知硬件 -->
+    <!-- LiDAR -->
+    <link name="laser_link">
+        <visual>
+            <origin xyz="0.0 0.0 0.0" rpy="0.0 0.0 0.0" />
+            <geometry>
+                <cylinder radius="0.05" length="0.05" />
+            </geometry>
+            <material name="blue">
+                <color rgba="0.0 0.0 1.0 1.0" />
+            </material>
+        </visual>
+        <collision>
+            <geometry>
+                <cylinder radius="0.05" length="0.05" />
+            </geometry>
+        </collision>
+        <xacro:cylinder_inertia m="0.1" r="0.05" h="0.05" />
+    </link>
+    <!-- GazeboLiDAR插件 -->
+    <gazebo reference="laser_link">
+        <sensor name="rplidar" type="ray">
+            <always_on>true</always_on>
+            <visualize>false</visualize>
+            <update_rate>10.0</update_rate>
+            <ray>
+                <scan>
+                    <horizontal>
+                        <samples>640</samples>
+                        <resolution>1</resolution>
+                        <min_angle>-3.1415926</min_angle>
+                        <max_angle>3.1415926</max_angle>
+                    </horizontal>
+                    <vertical>
+                        <samples>16</samples>
+                        <resolution>1</resolution>
+                        <min_angle>-0.26</min_angle>
+                        <max_angle>0.26</max_angle>
+                    </vertical>
+                </scan>
+                <range>
+                    <min>0.15</min>
+                    <max>120.0</max>
+                    <resolution>0.01</resolution>
+                </range>
+                <noise>
+                    <type>gaussian</type>
+                    <mean>0.0</mean>
+                    <stddev>0.01</stddev>
+                </noise>
+            </ray>
+            <plugin name="gazebo_ros_ray_sensor" filename="libgazebo_ros_ray_sensor.so">
+                <ros>
+                    <remapping>~/out:=points_raw</remapping>
+                </ros>
+                <output_type>sensor_msgs/PointCloud2</output_type>
+                <frame_name>laser_link</frame_name>
+            </plugin>
+        </sensor>
+    </gazebo>
+    <!-- 雷达增高架 -->
+    <!-- 参数 -->
+    <xacro:property name="support_radius" default="0.01" />
+    <xacro:property name="support_length" default="0.25" />
+    <xacro:property name="support_x_offset" default="${car_length/2 - 0.35}" />
+    <link name="laser_support_link">
+        <visual>
+            <geometry>
+                <cylinder radius="${support_radius}" length="${support_length}" />
+            </geometry>
+            <material name="gray">
+                <color rgba="0.5 0.5 0.5 1.0" />
+            </material>
+        </visual>
+        <collision>
+            <geometry>
+                <cylinder radius="${support_radius}" length="${support_length}" />
+            </geometry>
+        </collision>
+        <xacro:cylinder_inertia m="0.2" r="0.01" h="0.25" />
+    </link>
+    <joint name="support_joint" type="fixed">
+        <parent link="base_link" />
+        <child link="laser_support_link" />
+        <origin xyz="${support_x_offset} 0 ${car_height/2 + support_length/2}" rpy="0.0 0.0 0.0" />
+    </joint>
+    <joint name="laser_joint" type="fixed">
+        <parent link="laser_support_link" />
+        <child link="laser_link" />
+        <origin xyz="0.0 0.0 ${support_length/2 + 0.025}" />
+    </joint>
+    <!-- IMU -->
+    <link name="imu_link">
+        <visual>
+            <geometry>
+                <box size="0.02 0.02 0.01" />
+            </geometry>
+            <material name="orange">
+                <color rgba="1.0 0.5 0.0 1.0" />
+            </material>
+        </visual>
+        <xacro:box_inertia m="0.01" w="0.02" h="0.02" d="0.01" />
+    </link>
+    <joint name="imu_joint" type="fixed">
+        <parent link="base_link" />
+        <child link="imu_link" />
+        <origin xyz="0.0 0.0 0.0" rpy="0.0 0.0 0.0" />
+    </joint>
+    <!-- Gazebo IMU 插件-->
+    <gazebo reference="imu_link">
+        <sensor name="imu_sensor" type="imu">
+            <always_on>true</always_on>
+            <update_rate>100.0</update_rate>
+            <imu>
+                <!-- 角速度噪音 -->
+                <angular_velocity>
+                    <x>
+                        <noise type="gaussian">
+                            <mean>0.0</mean>  <!-- 噪声均值 -->
+                            <stddev>2e-4</stddev> <!-- 标准差：0.0002 rad/s-->
+                        </noise>
+                    </x>
+                    <y>
+                        <noise type="gaussian">
+                            <mean>0.0</mean>  <!-- 噪声均值 -->
+                            <stddev>2e-4</stddev> <!-- 标准差：0.0002 rad/s-->
+                        </noise>
+                    </y>
+                    <z>
+                        <noise type="gaussian">
+                            <mean>0.0</mean>  <!-- 噪声均值 -->
+                            <stddev>2e-4</stddev> <!-- 标准差：0.0002 rad/s-->
+                        </noise>
+                    </z>
+                </angular_velocity>
+                <!-- 线速度噪音（单位：m/s^2） -->
+                <linear_acceleration>
+                    <x>
+                        <noise type="gaussian">
+                            <mean>0.0</mean>  <!-- 噪声均值 -->
+                            <stddev>1.7e-4</stddev> <!-- 标准差：0.017 m/s^2-->
+                        </noise>
+                    </x>
+                    <y>
+                        <noise type="gaussian">
+                            <mean>0.0</mean>  <!-- 噪声均值 -->
+                            <stddev>1.7e-4</stddev> <!-- 标准差：0.017 m/s^2-->
+                        </noise>
+                    </y>
+                    <z>
+                        <noise type="gaussian">
+                            <mean>0.0</mean>  <!-- 噪声均值 -->
+                            <stddev>1.7e-4</stddev> <!-- 标准差：0.017 m/s^2-->
+                        </noise>
+                    </z>
+                </linear_acceleration>
+            </imu>
+            <plugin name="imu_plugin" filename="libgazebo_ros_imu_sensor.so">
+                <ros>
+                    <remapping>~/out:=imu</remapping>
+                </ros>
+                <frame_name>imu_link</frame_name>
+                <!-- 初始姿态偏置，通常设为全0 -->
+                <initial_orientation_as_reference>false</initial_orientation_as_reference>
+            </plugin>
+        </sensor>
+    </gazebo>
 </robot>
