Commit message: feat:完成RGBD搭建

File: src/aicar_simulation/urdf/aicar.urdf.xacro (robot description, xacro)
@@ -367,3 +367,79 @@
         </sensor>
     </gazebo>
+    <!-- RGB-D 相机组件 -->
+    <!-- 相机尺寸参数（参考Realsense D435） -->
+    <xacro:property name="camera_length" default="0.03" /> <!-- X方向深度 -->
+    <xacro:property name="camera_width" default="0.10" />  <!-- Y方向深度 -->
+    <xacro:property name="camera_height" default="0.03" />  <!-- Z方向深度 -->
+    <!-- 相机物理外壳 -->
+    <link name="camera_link">
+        <visual>
+            <geometry>
+                <box size="${camera_length} ${camera_width} ${camera_height}" />
+            </geometry>
+            <material name="black">
+                <color rgba="0.0 0.0 0.0 1.0" />
+            </material>
+        </visual>
+        <collision>
+            <geometry>
+                <box size="${camera_length} ${camera_width} ${camera_height}" />
+            </geometry>
+        </collision>
+        <xacro:box_inertia m="0.1" w="${camera_width}" h="${camera_height}" d="${camera_length}" />
+    </link>
+    <!-- 相机安装到车上 -->
+    <joint name="camera_joint" type="fixed">
+        <parent link="base_link" />
+        <child link="camera_link" />
+        <!-- 安装位置：车头最前端 -->
+        <origin xyz="${car_length/2} 0.0 ${car_height/2 + camera_height/2}" />
+    </joint>
+    <!-- 光学坐标系转换（解决点云歪斜问题） -->
+    <!-- 虚拟link,提负责提供坐标定义 -->
+    <link name="camera_optical_frame" />
+    <joint name="camera_optical_joint" type="fixed">
+        <parent link="camera_link" />
+        <child link="camera_optical_frame" />
+        <!--
+                旋转逻辑：
+                RGB-D 坐标系 Z前 X右 Y下， 对齐   旋转顺序是ZYX
+                1. 绕Z轴旋转-90度（-pi/2）： 此时： Y前 X右 Z上
+                2. 绕X轴旋转-90度（-pi/2）： 此时： Z前 X右 Y下
+            -->
+        <origin xyz="0.0 0.0 0.0" rpy="${-pi/2} 0.0 ${-pi/2}"/>
+    </joint>
+    <gazebo reference="camera_link">
+        <!-- sensor 类型必须是 depth -->
+        <sensor name="camera_sensor" type="depth">
+            <always_on>true</always_on>
+            <update_rate>30.0</update_rate>
+            <camera>
+                <horizontal_fov>1.50098</horizontal_fov> <!-- 水平视角，越86度 -->
+                <image>
+                    <width>640</width>
+                    <height>480</height>
+                    <format>R8G8B8</format>
+                </image>
+                <clip>
+                    <near>0.1</near> <!-- 最近看10厘米 -->
+                    <far>10.0</far> <!-- 最远看100米 -->
+                </clip>
+            </camera>
+            <plugin name="camera_plugin" filename="libgazebo_ros_camera.so">
+                <ros>
+                    <!-- 将默认话题名重映射成更规范的名称 -->
+                    <remapping>custom_camera/image_raw:=camera/color/image_raw</remapping>
+                    <remapping>custom_camera/image_depth:=camera/depth/image_raw</remapping>
+                    <remapping>custom_camera/camera_info:=camera/camera_info</remapping>
+                    <remapping>custom_camera/points:=camera/depth/points</remapping>
+                </ros>
+                <!-- 关键：必须绑定到刚才旋转后的坐标系 -->
+                <frame_name>camera_optical_frame</frame_name>
+                <!-- 深度数据相关参数 -->
+                <min_depth>0.1</min_depth>
+                <max_depth>10.0</max_depth>
+            </plugin>
+        </sensor>
+    </gazebo>
 </robot>
